File: Taito System SJ/KiCAD/CPUPC2.kicad_sch (KiCad schematic)
At the start: 15 parts, among them U32 74LS367, U35 74LS32, U45 74LS367, U7 74LS374, U8 74LS374, U9 74LS173

Commit message: Added CPU
Parts:
- removed U32, U45: 74LS367, symbol jt74:74LS367
- removed U35, U? (x4): 74LS32, symbol jt74:74LS32
- removed U7, U8: 74LS374, symbol jt74:74LS374
- removed U9: 74LS173, symbol jt74:74LS173
- removed U? (x3): 74LS138, symbol jt74:74LS138
- removed U?, U??: 74LS04, symbol jt74:74LS04
