File: Taito System SJ/KiCAD/CPUPC1.kicad_sch (KiCad schematic)
At the start: 42 parts, among them U11 74LS161, U12 74LS10, U13 74LS161, U17 74LS85, U18 74LS85, U19 74LS85, U21 74LS04, U22 74LS86, U24 74LS161, U25 74LS86, U26 74LS161, U34 74LS08, U36 74LS04, U37 74LS164, U38 74LS175, U51 74LS74, U61 74LS02, U62 74LS00, U63 74LS367, U74 74LS74, U75 74LS74, U88 74LS04, U94 74LS32, U95 74LS04, U97 74LS74

Commit message: Multiple updates while coding core
Parts:
- gave numbers to parts that had none: 1
Connections:
- net H31: no longer U17.10 (A0), U18.10 (A0)
- net H32: no longer U17.12 (A1), U18.12 (A1)
- net H33: no longer U17.13 (A2), U18.13 (A2)
- new net H11: U17.10 (A0)
- new net H12: U17.12 (A1)
- new net H13: U17.13 (A2)
- new net H21: U18.10 (A0)
- new net H22: U18.12 (A1)
- new net H23: U18.13 (A2)
Changed lines of the file:
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@@
     (effects (font (size 1.27 1.27)) (justify right bottom))
   )
-  (label "H32" (at 453.39 128.27 180) (fields_autoplaced)
+  (label "H22" (at 453.39 128.27 180) (fields_autoplaced)
     (effects (font (size 1.27 1.27)) (justify right bottom))
   )
@@
     (effects (font (size 1.27 1.27)) (justify right bottom))
   )
-  (label "H31" (at 453.39 173.99 180) (fields_autoplaced)
+  (label "H11" (at 453.39 173.99 180) (fields_autoplaced)
     (effects (font (size 1.27 1.27)) (justify right bottom))
   )
@@
     (effects (font (size 1.27 1.27)) (justify left bottom))
   )
-  (label "H32" (at 453.39 171.45 180) (fields_autoplaced)
+  (label "H12" (at 453.39 171.45 180) (fields_autoplaced)
     (effects (font (size 1.27 1.27)) (justify right bottom))
   )
@@
     (effects (font (size 1.27 1.27)) (justify left bottom))
   )
-  (label "H33" (at 453.39 125.73 180) (fields_autoplaced)
+  (label "H23" (at 453.39 125.73 180) (fields_autoplaced)
     (effects (font (size 1.27 1.27)) (justify right bottom))
   )
@@
     (effects (font (size 1.27 1.27)) (justify right bottom))
   )
-  (label "H33" (at 453.39 168.91 180) (fields_autoplaced)
+  (label "H13" (at 453.39 168.91 180) (fields_autoplaced)
     (effects (font (size 1.27 1.27)) (justify right bottom))
   )
@@
     (effects (font (size 1.27 1.27)) (justify right bottom))
   )
-  (label "H31" (at 453.39 130.81 180) (fields_autoplaced)
+  (label "H21" (at 453.39 130.81 180) (fields_autoplaced)
     (effects (font (size 1.27 1.27)) (justify right bottom))
   )
@@
   (symbol (lib_id "jt74:74LS04") (at 519.43 130.81 0) (unit 4)
     (in_bom yes) (on_board yes) (dnp no) (fields_autoplaced)
-    (property "Reference" "U?" (at 519.43 123.3002 0)
-      (effects (font (size 1.27 1.27)))
-    )
-    (property "Value" "74LS04" (at 519.43 125.8371 0)
+    (property "Reference" "U21" (at 519.43 123.19 0)
+      (effects (font (size 1.27 1.27)))
+    )
+    (property "Value" "74LS04" (at 519.43 125.73 0)
       (effects (font (size 1.27 1.27)))
     )
@@
       (project "TAITOSJ"
         (path "/c9398d89-67dd-4ff5-9367-82e2b6879830/4965ed65-3406-4c92-8365-069f7161183c"
-          (reference "U?") (unit 4)
+          (reference "U21") (unit 4)
         )
       )
@@
   (symbol (lib_id "jt74:74LS04") (at 519.43 86.36 0) (unit 1)
     (in_bom yes) (on_board yes) (dnp no) (fields_autoplaced)
-    (property "Reference" "U?" (at 519.43 78.8502 0)
-      (effects (font (size 1.27 1.27)))
-    )
-    (property "Value" "74LS04" (at 519.43 81.3871 0)
+    (property "Reference" "U21" (at 519.43 78.74 0)
+      (effects (font (size 1.27 1.27)))
+    )
+    (property "Value" "74LS04" (at 519.43 81.28 0)
       (effects (font (size 1.27 1.27)))
     )
@@
       (project "TAITOSJ"
         (path "/c9398d89-67dd-4ff5-9367-82e2b6879830/4965ed65-3406-4c92-8365-069f7161183c"
-          (reference "U?") (unit 1)
+          (reference "U21") (unit 1)
         )
       )
@@
   (symbol (lib_id "jt74:74LS04") (at 519.43 173.99 0) (unit 5)
     (in_bom yes) (on_board yes) (dnp no) (fields_autoplaced)
-    (property "Reference" "U?" (at 519.43 166.4802 0)
-      (effects (font (size 1.27 1.27)))
-    )
-    (property "Value" "74LS04" (at 519.43 169.0171 0)
+    (property "Reference" "U21" (at 519.43 166.37 0)
+      (effects (font (size 1.27 1.27)))
+    )
+    (property "Value" "74LS04" (at 519.43 168.91 0)
       (effects (font (size 1.27 1.27)))
     )
@@
       (project "TAITOSJ"
         (path "/c9398d89-67dd-4ff5-9367-82e2b6879830/4965ed65-3406-4c92-8365-069f7161183c"
-          (reference "U?") (unit 5)
-        )
-      )
+          (reference "U21") (unit 5)
+        )
+      )
