File: Taito System SJ/KiCAD/ROMBOARD5.kicad_sch (KiCad schematic)
At the start: 13 parts, among them U1-ROM1 M2732, U10 40193, U11 40193, U12 40193, U13 40193, U2-ROM2 M2732, U3-ROM3 M2732, U4-ROM4 M2732, U5-ROM5 M2732, U6-ROM6 M2732, U7-ROM7 M2732, U8-ROM8 M2732, U9 74LS138

Commit message: Start of gameboard
Parts:
- removed U10, U11, U12, U13: 40193, symbol 4xxx_IEEE:40193
- added U10, U11, U12, U13: 74LS193, symbol jt74:74LS193
Connections:
- net DATABUS_D0: now also U10.15 (P0), U11.15 (P0)
- net DATABUS_D1: now also U10.1 (P1), U11.1 (P1)
- net DATABUS_D2: now also U10.10 (P2), U11.10 (P2)
- net DATABUS_D3: now also U10.9 (P3), U11.9 (P3)
- net DATABUS_D4: now also U12.15 (P0), U13.15 (P0)
- net DATABUS_D5: now also U12.1 (P1), U13.1 (P1)
- net DATABUS_D6: now also U12.10 (P2), U13.10 (P2)
- net DATABUS_D7: now also U12.9 (P3), U13.9 (P3)
- net EXTROM1: now also U10.11 (Pl), U12.11 (Pl)
- net EXTROM2: now also U11.11 (Pl), U13.11 (Pl)
- net EXT_ADDR_A0: now also U10.3 (Q0)
- net EXT_ADDR_A1: now also U10.2 (Q1)
- net EXT_ADDR_A10: now also U11.6 (Q2)
- net EXT_ADDR_A11: now also U11.7 (Q3)
- net EXT_ADDR_A12: now also U13.3 (Q0)
- net EXT_ADDR_A13: now also U13.2 (Q1)
- net EXT_ADDR_A14: now also U13.6 (Q2)
- net EXT_ADDR_A15: now also U13.7 (Q3)
- net EXT_ADDR_A2: now also U10.6 (Q2)
- net EXT_ADDR_A3: now also U10.7 (Q3)
- net EXT_ADDR_A4: now also U12.3 (Q0)
- net EXT_ADDR_A5: now also U12.2 (Q1)
- net EXT_ADDR_A6: now also U12.6 (Q2)
- net EXT_ADDR_A7: now also U12.7 (Q3)
- net EXT_ADDR_A8: now also U11.3 (Q0)
- net EXT_ADDR_A9: now also U11.2 (Q1)
- net VCC: now also U10.4 (CpDw), U11.4 (CpDw), U12.4 (CpDw), U13.4 (CpDw)
- net ~{EXRHR}: now also U10.5 (CpUp)
- net GNDPWR: now reaches U9.6 (E3)
- net GNDPWR: now also U10.14 (Mr), U11.14 (Mr), U12.14 (Mr), U13.14 (Mr)
- new net: U11.5 (CpUp), U12.12 (TcUp)
- new net: U10.8 (GND), U12.16 (VCC)
- new net: U10.12 (TcUp), U12.5 (CpUp)
- new net: U11.12 (TcUp), U13.5 (CpUp)
- new net: U11.8 (GND), U13.16 (VCC)

Commit message: Multiple updates while coding core
Connections:
- net GNDPWR: no longer U9.6 (E3)
- net VCC: now also U9.6 (E3)
Changed lines of the file:
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@@
-    (stroke (width 0) (type default))
-  )
-  (wire (pts (xy 146.05 227.33) (xy 143.51 227.33))
     (stroke (width 0) (type default))
   )
@@
     (stroke (width 0) (type default))
   )
-  (wire (pts (xy 143.51 227.33) (xy 143.51 228.6))
-    (stroke (width 0) (type default))
-  )
   (wire (pts (xy 237.49 213.36) (xy 237.49 214.63))
     (stroke (width 0) (type default))
@@
   )
   (wire (pts (xy 50.8 101.6) (xy 74.93 101.6))
+    (stroke (width 0) (type default))
+  )
+  (wire (pts (xy 140.97 227.33) (xy 146.05 227.33))
     (stroke (width 0) (type default))
   )
@@
     )
   )
-  (symbol (lib_id "power:GNDPWR") (at 143.51 228.6 0) (unit 1)
-    (in_bom yes) (on_board yes) (dnp no) (fields_autoplaced)
-    (property "Reference" "#PWR?" (at 143.51 233.68 0)
-      (effects (font (size 1.27 1.27)) hide)
-    )
-    (property "Value" "GNDPWR" (at 143.383 232.637 0)
-      (effects (font (size 1.27 1.27)))
-    )
-    (property "Footprint" "" (at 143.51 229.87 0)
-      (effects (font (size 1.27 1.27)) hide)
-    )
-    (property "Datasheet" "" (at 143.51 229.87 0)
-      (effects (font (size 1.27 1.27)) hide)
-    )
-    (pin "1")
-    (instances
-      (project "TAITOSJ"
-        (path "/c9398d89-67dd-4ff5-9367-82e2b6879830/34ec39bd-d7df-4ca2-9130-4c3bb5b8903a"
-          (reference "#PWR?") (unit 1)
-        )
-      )
-    )
-  )
   (symbol (lib_id "arcade:M2732AF1") (at 248.92 55.88 0) (unit 1)
     (in_bom yes) (on_board yes) (dnp no) (fields_autoplaced)
@@
         )
       )
+    )
+  )
+  (symbol (lib_name "VCC_1") (lib_id "power:VCC") (at 140.97 227.33 90) (unit 1)
+    (in_bom yes) (on_board yes) (dnp no) (fields_autoplaced)
+    (property "Reference" "#PWR013" (at 144.78 227.33 0)
+      (effects (font (size 1.27 1.27)) hide)
+    )
+    (property "Value" "VCC" (at 137.16 227.965 90)
+      (effects (font (size 1.27 1.27)) (justify left))
+    )
+    (property "Footprint" "" (at 140.97 227.33 0)
+      (effects (font (size 1.27 1.27)) hide)
+    )
+    (property "Datasheet" "" (at 140.97 227.33 0)
+      (effects (font (size 1.27 1.27)) hide)
+    )
+    (pin "1")
+    (instances
+      (project "TAITOSJ"
+        (path "/c9398d89-67dd-4ff5-9367-82e2b6879830/34ec39bd-d7df-4ca2-9130-4c3bb5b8903a"
+          (reference "#PWR013") (unit 1)
+        )
+      )
