File: Taito System SJ/KiCAD/VB1.kicad_sch (KiCad schematic)
At the start: 60 parts, among them U101 74LS00, U102 74LS367, U103 74LS367, U104 RAM_2016, U105 RAM_2016, U106 RAM_2016, U107 RAM_2016, U108 RAM_2016, U109 RAM_2016, U22 82S129 - EB16, U23 74LS157, U24 74LS374, U25 74LS153, U33 74LS27, U34 74LS374, U35 74LS174, U36 74LS174, U37 74LS153, U38 74LS153, U4 74LS04, U45 74LS367, U46 74LS166, U47 74LS273, U48 74LS27, U49 74LS166, U50 74LS273, U51 74LS253, U52 74LS166, U53 74LS273, U54 74LS10, U58 74LS32, U60 74LS166, U61 74LS273, U62 74LS157, U63 74LS166, U64 74LS273, U65 74LS157, U66 74LS166, U67 74LS273, U68 74LS157, U72 74LS08, U74 74LS166, U75 74LS273, U76 74LS157, U77 74LS166, U78 74LS273, U79 74LS157, U80 74LS166, U81 74LS273, U82 74LS157, U87 74LS08, U89 74LS166, U90 74LS367, U91 74LS08, U92 74LS166, U93 74LS367, U94 74LS367, U95 74LS166, U96 74LS367

Commit message: Multiple updates while coding core
Parts:
- added R?: ?, symbol Device:R_US
- added unit 1 of U54
- added unit 1 of U58
Connections:
- net CDR_RQ1 is gone; now on net CDR1RQ: U91.5
- net CDR_RQ2 is gone; now on net CDR2RQ: U91.1
- net CDR_RQ3 is gone; now on net CDR3RQ: U91.13
- net CDR_RQ4 is gone; now on net CDR4RQ: U87.9
- net CDR_RQ5 is gone; now on net CDR5RQ: U87.12
- net CDR_RQ6 is gone; now on net CDR6RQ: U87.1
- net CDRRQ: now also U104.20 (~{OE}), U105.20 (~{OE}), U106.20 (~{OE}), U107.20 (~{OE}), U108.20 (~{OE}), U109.20 (~{OE}), U58.1
- net CRD0: now also U68.14 (I0d); no longer U68.13 (I1d)
- net CRD1: now also U68.11 (I0c); no longer U68.10 (I1c)
- net CRD2: now also U68.5 (I0b); no longer U68.6 (I1b)
- net CRD3: now also U68.2 (I0a); no longer U68.3 (I1a)
- net CRD4: now also U68.3 (I1a); no longer U68.2 (I0a)
- net CRD5: now also U68.6 (I1b); no longer U68.5 (I0b)
- net CRD6: now also U68.10 (I1c); no longer U68.11 (I0c)
- net CRD7: now also U68.13 (I1d); no longer U68.14 (I0d)
- net MD23: no longer U25.3 (I3a), U33.1, U52.13 (Qh)
- net VCC: now also R?.1
- net SELVRAMB2: now reaches U101.12, U51.7 (Za), U91.12, U91.2, U91.4
- net SELVRAMB2: now also R?.2
- net at U104.21 (~{WE}), U105.21 (~{WE}), U106.21 (~{WE})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: now also U54.3
- net SELVRAM_B1: now reaches U101.11, U87.10, U87.13, U87.2
- net LDNLD: now reaches U58.11, U89.15 (PE), U92.15 (PE), U95.15 (PE)
- net Q2: now reaches U92.13 (Qh)
- net Q3: now reaches U89.13 (Qh)
- net Q1: now reaches U95.13 (Qh)
- net ~{PH34} renamed ~{PHA34}
- new net: U54.2, U58.3
- new net SN31: U25.3 (I3a), U33.1, U52.13 (Qh)
- new net ~{PH23}: U54.1
- new net ~{WR}: U58.2
Other:
- note added: "SELECT RAM BANK"

Commit message: Tidied up loose ends
Connections:
- net OBJ: now reaches U22.5 (A0), U48.6
- net SCN1: now reaches U22.6 (A1), U48.8
- net SCN2: now reaches U22.7 (A2), U48.6
- net SCN3: now reaches U22.4 (A3), U33.12
Changed lines of the file:
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@@
   (junction (at 365.76 633.73) (diameter 0) (color 0 0 0 0)
   )
+  (junction (at 320.04 775.97) (diameter 0) (color 0 0 0 0)
+  )
   (junction (at 149.86 431.8) (diameter 0) (color 0 0 0 0)
   )
@@
   (junction (at 149.86 434.34) (diameter 0) (color 0 0 0 0)
   )
+  (junction (at 320.04 745.49) (diameter 0) (color 0 0 0 0)
+  )
   (junction (at 284.48 450.85) (diameter 0) (color 0 0 0 0)
   )
@@
   (junction (at 363.22 163.83) (diameter 0) (color 0 0 0 0)
   )
+  (junction (at 320.04 760.73) (diameter 0) (color 0 0 0 0)
+  )
   (junction (at 494.03 563.88) (diameter 0) (color 0 0 0 0)
   )
@@
   (junction (at 365.76 295.91) (diameter 0) (color 0 0 0 0)
   )
+  (junction (at 320.04 730.25) (diameter 0) (color 0 0 0 0)
+  )
   (junction (at 365.76 397.51) (diameter 0) (color 0 0 0 0)
   )
@@
     (stroke (width 0) (type default))
   )
+  (wire (pts (xy 320.04 775.97) (xy 337.82 775.97))
+    (stroke (width 0) (type default))
+  )
   (wire (pts (xy 99.06 218.44) (xy 99.06 269.24))
     (stroke (width 0) (type default))
@@
     (stroke (width 0) (type default))
   )
-  (wire (pts (xy 326.39 737.87) (xy 350.52 737.87))
+  (wire (pts (xy 337.82 737.87) (xy 350.52 737.87))
     (stroke (width 0) (type default))
   )
@@
     (stroke (width 0) (type default))
   )
-  (wire (pts (xy 326.39 775.97) (xy 326.39 737.87))
+  (wire (pts (xy 337.82 775.97) (xy 337.82 737.87))
     (stroke (width 0) (type default))
   )
@@
     (stroke (width 0) (type default))
   )
-  (wire (pts (xy 323.85 735.33) (xy 350.52 735.33))
+  (wire (pts (xy 335.28 735.33) (xy 350.52 735.33))
     (stroke (width 0) (type default))
   )
@@
     (stroke (width 0) (type default))
   )
+  (wire (pts (xy 320.04 745.49) (xy 332.74 745.49))
+    (stroke (width 0) (type default))
+  )
   (wire (pts (xy 370.84 745.49) (xy 370.84 748.03))
     (stroke (width 0) (type default))
@@
     (stroke (width 0) (type default))
   )
-  (wire (pts (xy 321.31 732.79) (xy 350.52 732.79))
+  (wire (pts (xy 332.74 732.79) (xy 350.52 732.79))
     (stroke (width 0) (type default))
   )
@@
     (stroke (width 0) (type default))
   )
+  (wire (pts (xy 320.04 758.19) (xy 320.04 760.73))
+    (stroke (width 0) (type default))
+  )
   (wire (pts (xy 303.53 557.53) (xy 273.05 557.53))
     (stroke (width 0) (type default))
@@
     (stroke (width 0) (type default))
   )
-  (wire (pts (xy 318.77 775.97) (xy 326.39 775.97))
+  (wire (pts (xy 318.77 775.97) (xy 320.04 775.97))
     (stroke (width 0) (type default))
   )
@@
     (stroke (width 0) (type default))
   )
+  (wire (pts (xy 322.58 773.43) (xy 320.04 773.43))
+    (stroke (width 0) (type default))
+  )
   (bus (pts (xy 407.67 506.73) (xy 407.67 557.53))
     (stroke (width 0) (type default))
@@
     (stroke (width 0) (type default))
   )
-  (wire (pts (xy 318.77 760.73) (xy 323.85 760.73))
+  (wire (pts (xy 318.77 760.73) (xy 320.04 760.73))
     (stroke (width 0) (type default))
   )
@@
     (stroke (width 0) (type default))
   )
-  (wire (pts (xy 318.77 745.49) (xy 321.31 745.49))
+  (wire (pts (xy 318.77 745.49) (xy 320.04 745.49))
     (stroke (width 0) (type default))
   )
@@
     (stroke (width 0) (type default))
   )
+  (wire (pts (xy 322.58 742.95) (xy 320.04 742.95))
+    (stroke (width 0) (type default))
+  )
   (wire (pts (xy 434.34 434.34) (xy 431.8 434.34))
     (stroke (width 0) (type default))
@@
     (stroke (width 0) (type default))
   )
+  (wire (pts (xy 320.04 730.25) (xy 350.52 730.25))
+    (stroke (width 0) (type default))
+  )
   (wire (pts (xy 300.99 499.11) (xy 303.53 499.11))
     (stroke (width 0) (type default))
@@
     (stroke (width 0) (type default))
   )
-  (wire (pts (xy 318.77 730.25) (xy 350.52 730.25))
+  (wire (pts (xy 318.77 730.25) (xy 320.04 730.25))
     (stroke (width 0) (type default))
   )
@@
     (stroke (width 0) (type default))
   )
+  (wire (pts (xy 322.58 727.71) (xy 320.04 727.71))
+    (stroke (width 0) (type default))
+  )
   (wire (pts (xy 99.06 269.24) (xy 101.6 269.24))
     (stroke (width 0) (type default))
@@
     (stroke (width 0) (type default))
   )
-  (wire (pts (xy 323.85 760.73) (xy 323.85 735.33))
+  (wire (pts (xy 335.28 760.73) (xy 335.28 735.33))
     (stroke (width 0) (type default))
   )
@@
     (stroke (width 0) (type default))
   )
+  (wire (pts (xy 320.04 773.43) (xy 320.04 775.97))
+    (stroke (width 0) (type default))
+  )
   (wire (pts (xy 177.8 668.02) (xy 184.15 668.02))
     (stroke (width 0) (type default))
@@
     (stroke (width 0) (type default))
   )
+  (wire (pts (xy 320.04 760.73) (xy 335.28 760.73))
+    (stroke (width 0) (type default))
+  )
   (bus (pts (xy 407.67 601.98) (xy 407.67 604.52))
     (stroke (width 0) (type default))
@@
     (stroke (width 0) (type default))
   )
+  (wire (pts (xy 320.04 727.71) (xy 320.04 730.25))
+    (stroke (width 0) (type default))
+  )
   (wire (pts (xy 303.53 140.97) (xy 273.05 140.97))
     (stroke (width 0) (type default))
@@
     (stroke (width 0) (type default))
   )
-  (wire (pts (xy 321.31 745.49) (xy 321.31 732.79))
+  (wire (pts (xy 332.74 745.49) (xy 332.74 732.79))
     (stroke (width 0) (type default))
   )
@@
     (stroke (width 0) (type default))
   )
+  (wire (pts (xy 320.04 742.95) (xy 320.04 745.49))
+    (stroke (width 0) (type default))
+  )
   (bus (pts (xy 420.37 478.79) (xy 420.37 481.33))
     (stroke (width 0) (type default))
@@
     (stroke (width 0) (type default))
   )
+  (wire (pts (xy 322.58 758.19) (xy 320.04 758.19))
+    (stroke (width 0) (type default))
+  )
   (wire (pts (xy 99.06 269.24) (xy 99.06 271.78))
     (stroke (width 0) (type default))
@@
     )
   )
+  (global_label "SCN2" (shape output) (at 322.58 758.19 0) (fields_autoplaced)
+    (effects (font (size 1.27 1.27)) (justify left))
+    (property "Intersheetrefs" "${INTERSHEET_REFS}" (at 330.5053 758.19 0)
+      (effects (font (size 1.27 1.27)) (justify left) hide)
+    )
+  )
   (global_label "~{SN2OFF}" (shape input) (at 360.68 354.33 180) (fields_autoplaced)
     (effects (font (size 1.27 1.27)) (justify right))
@@
     )
   )
+  (global_label "OBJ" (shape output) (at 322.58 727.71 0) (fields_autoplaced)
+    (effects (font (size 1.27 1.27)) (justify left))
+    (property "Intersheetrefs" "${INTERSHEET_REFS}" (at 329.0539 727.71 0)
+      (effects (font (size 1.27 1.27)) (justify left) hide)
+    )
+  )
   (global_label "CDR6RQ" (shape input) (at 176.53 608.33 0) (fields_autoplaced)
     (effects (font (size 1.27 1.27)) (justify left))
@@
     )
   )
+  (global_label "SCN1" (shape output) (at 322.58 742.95 0) (fields_autoplaced)
+    (effects (font (size 1.27 1.27)) (justify left))
+    (property "Intersheetrefs" "${INTERSHEET_REFS}" (at 330.5053 742.95 0)
+      (effects (font (size 1.27 1.27)) (justify left) hide)
+    )
+  )
   (global_label "MA1" (shape output) (at 514.35 786.13 0) (fields_autoplaced)
     (effects (font (size 1.27 1.27)) (justify left))
@@
     )
   )
+  (global_label "SCN3" (shape output) (at 322.58 773.43 0) (fields_autoplaced)
+    (effects (font (size 1.27 1.27)) (justify left))
+    (property "Intersheetrefs" "${INTERSHEET_REFS}" (at 330.5053 773.43 0)
+      (effects (font (size 1.27 1.27)) (justify left) hide)
+    )
+  )

Commit message: Added MCU to Taito SJ Schematics
Other:
- note added: "CCHx CCH = CHARACTER BANK x = ASSOCIATED TILEMAP"
- note added: "MDxy MD = TILEMAP COLOR CODE x = TILEMAP # (1,2 or 3) y = COLOUR CODE"
- note added: "SNxy SN = TILEMAP DATA x = ASSOCIATED TILEMAP y = GRAPHIC BIT (3 BIT = 8 COLORS PER TILE)"
