File: Taito System SJ/KiCAD/VB2.kicad_sch (KiCad schematic)
At the start: 32 parts, among them U100 74LS367, U101 74LS00, U12 74LS02, U16 74LS367, U17 NEC_UPD2114, U18 NEC_UPD2114, U19 74LS32, U20 74LS157, U21 74LS157, U26 74LS139, U3 74LS367, U30 74LS367, U31 74LS367, U32 74LS273, U39 74LS32, U4 74LS04, U44 74LS86, U58 74LS32, U59 74LS32, U73 74LS139, U83 74LS273, U83 74LS83, U85 74LS175, U86 74LS86, U88 74LS175, U98 74LS83, U99 74LS374

Commit message: Update before transfer
Parts:
- U32: value 74LS273 -> 74LS96
Connections:
- net D0: no longer U32.18 (D7)
- net D1: no longer U32.17 (D6)
- net D2: now also U32.9 (SER); no longer U32.14 (D5)
- net D3: now also U32.2 (P0); no longer U32.13 (D4)
- net D4: now also U32.3 (P1); no longer U32.8 (D3)
- net D5: now also U32.4 (P2); no longer U32.7 (D2)
- net D6: now also U32.6 (P3); no longer U32.4 (D1)
- net D7: now also U32.7 (P4); no longer U32.3 (D0)
- net GND: now also U32.12 (GND)
- net OBJEX: no longer U32.15 (Q5)
- net VCC: now also U32.5 (VCC); no longer U32.1 (~{Mr})
- net ~{OBJOFF}: now also U32.10 (Q4); no longer U32.2 (Q0)
- net ~{SN1OFF}: now also U32.14 (Q1); no longer U32.9 (Q3)
- net ~{SN2OFF}: now also U32.13 (Q2); no longer U32.6 (Q2)
- net ~{SN3OFF}: now also U32.11 (Q3); no longer U32.5 (Q1)
- net ~{SOFF}: no longer U32.11 (Cp)
- net at U88.4 (D0): no longer U32.19 (Q7)
- net at U88.5 (D1): no longer U32.16 (Q6)

Commit message: Multiple updates while coding core
Parts:
- removed U32: 74LS96, symbol jt74:74LS273
- added U32: 74LS273, symbol 74xx:74LS273
Connections:
- net CHA0: now also U100.5 (O2a); no longer U100.7 (O3a)
- net CHA1: now also U100.7 (O3a); no longer U100.5 (O2a)
- net CHA2: now also U100.9 (O4a); no longer U100.3 (O1a)
- net CINV: now also U100.3 (O1a); no longer U100.9 (O4a)
- net D0: now also U32.18 (D7)
- net D1: now also U32.17 (D6)
- net D2: now also U32.14 (D5)
- net D3: now also U32.13 (D4)
- net D4: now also U32.8 (D3)
- net D5: now also U32.7 (D2)
- net D6: now also U32.4 (D1)
- net D7: now also U32.3 (D0)
- net OBJEX: now also U32.15 (Q5)
- net OD0: now also U85.4 (D0); no longer U85.12 (D2)
- net OD1: now also U85.5 (D1); no longer U85.13 (D3)
- net OD2: now also U85.12 (D2); no longer U85.4 (D0)
- net OD3: now also U85.13 (D3); no longer U85.5 (D1)
- net OMD1: now also U85.10 (Q2)
- net VCC: now also U32.1 (~{Mr})
- net ~{OBJOFF}: now also U32.2 (Q0)
- net ~{SN1OFF}: now also U32.9 (Q3)
- net ~{SN2OFF}: now also U32.6 (Q2)
- net ~{SN3OFF}: now also U32.5 (Q1)
- net ~{SOFF}: now also U32.11 (Cp)
- net ~{SRAMRQ}: now also U73.12 (O0); no longer U73.11 (O1)
- net at U88.4 (D0): now also U32.19 (Q7)
- net at U88.5 (D1): now also U32.16 (Q6)
- net at U83.15 (S4): now also U83.8 (D3); no longer U83.14 (D5)
- net at U83.2 (S3): now also U83.7 (D2); no longer U83.4 (D1)
- net at U83.6 (S2): now also U83.4 (D1); no longer U83.3 (D0)
- net at U83.9 (S1): now also U83.3 (D0); no longer U83.17 (D6)
- net at U83.12 (Q4): now also U86.13; no longer U86.9
- net at U86.9: now also U83.9 (Q3); no longer U83.15 (Q5)
- net at U83.16 (Q6): now also U86.10; no longer U44.2
- net at U98.2 (S3): now also U83.17 (D6); no longer U83.18 (D7)
- net at U83.19 (Q7): now also U86.9; no longer U86.13
- net at U83.2 (Q0): now also U44.1; no longer U86.1
- net at U86.4: now also U83.6 (Q2); no longer U83.5 (Q1)
- net at U98.15 (S4): now also U83.18 (D7); no longer U83.7 (D2)
- net at U98.6 (S2): now also U83.14 (D5); no longer U83.8 (D3)
- net at U86.12: now also U83.15 (Q5); no longer U83.9 (Q3)
- net OD1_PH7: now reaches U86.10, U86.2, U86.5
- net OD1_PH7: now also U100.2 (I1), U44.2, U85.7 (Q1); no longer U44.1, U85.15 (Q3)
- net at U86.6: now also U100.10 (I4); no longer U100.2 (I1)
- net at U44.3: now also U100.4 (I2); no longer U100.6 (I3)
- net OBJ_ADDR_EN: now reaches U100.1 (OEa), U100.15 (OEb), U58.8, U99.1 (~{OE})
- net at U86.3: now also U100.6 (I3); no longer U100.4 (I2)
- net OD0_PH7: now reaches U85.2 (Q0)
- net OD0_PH7: now also U86.13
- new net: U83.5 (Q1), U86.1
Other:
- note added: "P-15"
- note added: "SPRITE BANK SELECT"
- note added: "The original schematic shows connections to U8 going to the right pin, but the wrong input name. The input names make more sense, so for documentation of the FPGA core I have utilized the naming scheme."
- moved on the sheet: U44A, U86A, U86B, U86C, U86D, U99

Commit message: Tidied up loose ends
Parts:
- gave numbers to parts that had none: 5
Connections:
- net OD1_PH7: no longer U100.2 (I1)
- net VCC: now also U11.9 (~{MR}), U9.9 (~{MR})
- net HITON?? renamed HITON
- net HLD0 renamed HLP0
- net HLD1 renamed HLP1
- net HLD2 renamed HLP2
- net OD0_PH7 renamed OBJ_CINV
- net OBJ_CINV: now also U100.2 (I1)

Commit message: Added MCU to Taito SJ Schematics
Parts:
- renumbered U83 to U97
Connections:
- net GND: now also U32.10 (GND)
- net VCC: now also U32.20 (VCC)
