File: Taito System SJ/KiCAD/VB3.kicad_sch (KiCad schematic)
At the start: 30 parts, among them U13 74LS157, U14 74LS157, U15 74LS175, U19 74LS32, U2 74LS157, U27 74LS273, U28 74LS86, U29 74LS163, U33 74LS27, U39 74LS32, U4 74LS04, U40 74LS174, U41 RAM_5501, U42 74LS86, U43 74LS163, U5 74LS74, U54 74LS10, U55 74LS86, U56 74LS27, U57 74LS163, U6 74LS32, U69 RAM_5501, U7 74LS74, U70 74LS86, U71 74LS163, U72 74LS08

Commit message: Multiple updates while coding core
Parts:
- gave numbers to parts that had none: 2
- renumbered U2 to U1
Connections:
- net 16HN: now also U40.14 (D5)
- net 32HN: now also U40.13 (D4)
- net 64HN: now also U40.11 (D3)
- net CLK: now also U41.20 (WEn), U69.20 (WEn)
- net Q21': no longer U40.13 (D4)
- net Q22': no longer U40.14 (D5)
- net Q23': no longer U40.3 (D0), U40.4 (D1)
- net Q24': no longer U40.11 (D3)
- net ~{LNSL1}: now also U13.15 (E)
- net ~{LNSL2}: now also U1.15 (E)
- net OBJH: now reaches U13.1 (S)
- new net 128HN: U40.3 (D0)
- new net HBL: U40.4 (D1)
Changed lines of the file:
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@@
     (stroke (width 0) (type default))
   )
+  (wire (pts (xy 242.57 274.32) (xy 242.57 269.24))
+    (stroke (width 0) (type default))
+  )
   (wire (pts (xy 58.42 278.13) (xy 58.42 222.25))
     (stroke (width 0) (type default))
@@
     (stroke (width 0) (type default))
   )
+  (wire (pts (xy 194.31 336.55) (xy 201.93 336.55))
+    (stroke (width 0) (type default))
+  )
   (wire (pts (xy 261.62 43.18) (xy 233.68 43.18))
     (stroke (width 0) (type default))
@@
     (stroke (width 0) (type default))
   )
+  (wire (pts (xy 242.57 92.71) (xy 242.57 87.63))
+    (stroke (width 0) (type default))
+  )
   (wire (pts (xy 180.34 393.7) (xy 201.93 393.7))
     (stroke (width 0) (type default))
@@
     (stroke (width 0) (type default))
   )
-  (wire (pts (xy 190.5 334.01) (xy 201.93 334.01))
+  (wire (pts (xy 185.42 334.01) (xy 201.93 334.01))
     (stroke (width 0) (type default))
   )
@@
     (stroke (width 0) (type default))
   )
-  (wire (pts (xy 260.35 342.9) (xy 190.5 342.9))
+  (wire (pts (xy 260.35 342.9) (xy 185.42 342.9))
     (stroke (width 0) (type default))
   )
@@
     (stroke (width 0) (type default))
   )
+  (wire (pts (xy 194.31 152.4) (xy 201.93 152.4))
+    (stroke (width 0) (type default))
+  )
   (wire (pts (xy 66.04 86.36) (xy 99.06 86.36))
     (stroke (width 0) (type default))
@@
     (stroke (width 0) (type default))
   )
+  (wire (pts (xy 194.31 154.94) (xy 201.93 154.94))
+    (stroke (width 0) (type default))
+  )
   (wire (pts (xy 66.04 267.97) (xy 99.06 267.97))
     (stroke (width 0) (type default))
@@
     (stroke (width 0) (type default))
   )
-  (wire (pts (xy 190.5 342.9) (xy 190.5 334.01))
+  (wire (pts (xy 185.42 342.9) (xy 185.42 334.01))
     (stroke (width 0) (type default))
   )
@@
     (effects (font (size 1.27 1.27)) (justify left bottom))
   )
-  (label "Q21'" (at 351.79 330.2 0) (fields_autoplaced)
+  (label "32HN" (at 351.79 330.2 0) (fields_autoplaced)
     (effects (font (size 1.27 1.27)) (justify left bottom))
   )
@@
     (effects (font (size 1.27 1.27)) (justify left bottom))
   )
-  (label "Q24'" (at 351.79 332.74 0) (fields_autoplaced)
+  (label "64HN" (at 351.79 332.74 0) (fields_autoplaced)
     (effects (font (size 1.27 1.27)) (justify left bottom))
   )
@@
     (effects (font (size 1.27 1.27)) (justify left bottom))
   )
-  (label "Q22'" (at 351.79 327.66 0) (fields_autoplaced)
+  (label "16HN" (at 351.79 327.66 0) (fields_autoplaced)
     (effects (font (size 1.27 1.27)) (justify left bottom))
   )
@@
     (effects (font (size 1.27 1.27)) (justify left bottom))
   )
-  (label "Q23'" (at 351.79 340.36 0) (fields_autoplaced)
+  (label "128HN" (at 351.79 340.36 0) (fields_autoplaced)
     (effects (font (size 1.27 1.27)) (justify left bottom))
   )
@@
     (effects (font (size 1.27 1.27)) (justify left bottom))
   )
-  (label "Q23'" (at 351.79 337.82 0) (fields_autoplaced)
+  (label "HBL" (at 351.79 337.82 0) (fields_autoplaced)
     (effects (font (size 1.27 1.27)) (justify left bottom))
   )
@@
     )
   )
+  (global_label "CLK" (shape input) (at 242.57 92.71 270) (fields_autoplaced)
+    (effects (font (size 1.27 1.27)) (justify right))
+    (property "Intersheetrefs" "${INTERSHEET_REFS}" (at 242.57 99.1839 90)
+      (effects (font (size 1.27 1.27)) (justify right) hide)
+    )
+  )
   (global_label "~{PHA348}" (shape output) (at 499.11 236.22 0) (fields_autoplaced)
     (effects (font (size 1.27 1.27)) (justify left))
@@
     )
   )
+  (global_label "CLK" (shape input) (at 242.57 274.32 270) (fields_autoplaced)
+    (effects (font (size 1.27 1.27)) (justify right))
+    (property "Intersheetrefs" "${INTERSHEET_REFS}" (at 242.57 280.7939 90)
+      (effects (font (size 1.27 1.27)) (justify right) hide)
+    )
+  )
   (global_label "~{LNLD2}" (shape output) (at 499.11 227.33 0) (fields_autoplaced)
     (effects (font (size 1.27 1.27)) (justify left))
@@
     )
   )
+  (global_label "~{LNSL2}" (shape input) (at 194.31 336.55 180) (fields_autoplaced)
+    (effects (font (size 1.27 1.27)) (justify right))
+    (property "Intersheetrefs" "${INTERSHEET_REFS}" (at 185.5985 336.55 0)
+      (effects (font (size 1.27 1.27)) (justify right) hide)
+    )
+  )
   (global_label "H.INV" (shape input) (at 80.01 345.44 180) (fields_autoplaced)
     (effects (font (size 1.27 1.27)) (justify right))
@@
     )
   )
+  (global_label "OBJH" (shape input) (at 194.31 152.4 180) (fields_autoplaced)
+    (effects (font (size 1.27 1.27)) (justify right))
+    (property "Intersheetrefs" "${INTERSHEET_REFS}" (at 186.5056 152.4 0)
+      (effects (font (size 1.27 1.27)) (justify right) hide)
+    )
+  )
   (global_label "~{LNLD1}" (shape input) (at 55.88 109.22 180) (fields_autoplaced)
     (effects (font (size 1.27 1.27)) (justify right))
@@
     )
   )
+  (global_label "~{LNSL1}" (shape input) (at 194.31 154.94 180) (fields_autoplaced)
+    (effects (font (size 1.27 1.27)) (justify right))
+    (property "Intersheetrefs" "${INTERSHEET_REFS}" (at 186.0912 154.8606 0)
+      (effects (font (size 1.27 1.27)) (justify right) hide)
+    )
+  )
   (global_label "~{BLANK}" (shape input) (at 381 142.24 180) (fields_autoplaced)
     (effects (font (size 1.27 1.27)) (justify right))
@@
   (symbol (lib_id "jt74:74LS157") (at 214.63 322.58 0) (unit 1)
     (in_bom yes) (on_board yes) (dnp no) (fields_autoplaced)
-    (property "Reference" "U2" (at 214.63 303.7672 0)
+    (property "Reference" "U1" (at 214.63 303.53 0)
       (effects (font (size 1.27 1.27)))
     )
-    (property "Value" "74LS157" (at 214.63 306.3041 0)
+    (property "Value" "74LS157" (at 214.63 306.07 0)
       (effects (font (size 1.27 1.27)))
     )
@@
       (project "TAITOSJ"
         (path "/c9398d89-67dd-4ff5-9367-82e2b6879830/fa5496c1-bb75-4748-8ec7-34a2f42bf7c1"
-          (reference "U2") (unit 1)
+          (reference "U1") (unit 1)
         )
       )
@@
   (symbol (lib_id "jt74:74LS10") (at 361.95 203.2 0) (unit 3)
     (in_bom yes) (on_board yes) (dnp no) (fields_autoplaced)
-    (property "Reference" "U?" (at 361.95 195.6902 0)
+    (property "Reference" "U54" (at 361.9417 195.58 0)
       (effects (font (size 1.27 1.27)))
     )
-    (property "Value" "74LS10" (at 361.95 198.2271 0)
+    (property "Value" "74LS10" (at 361.9417 198.12 0)
       (effects (font (size 1.27 1.27)))
     )
@@
       (project "TAITOSJ"
         (path "/c9398d89-67dd-4ff5-9367-82e2b6879830/fa5496c1-bb75-4748-8ec7-34a2f42bf7c1"
-          (reference "U?") (unit 3)
+          (reference "U54") (unit 3)
         )
       )
@@
   (symbol (lib_id "jt74:74LS08") (at 97.79 161.29 0) (unit 3)
     (in_bom yes) (on_board yes) (dnp no) (fields_autoplaced)
-    (property "Reference" "U?" (at 97.79 153.7802 0)
+    (property "Reference" "U72" (at 97.7817 153.67 0)
       (effects (font (size 1.27 1.27)))
     )
-    (property "Value" "74LS08" (at 97.79 156.3171 0)
+    (property "Value" "74LS08" (at 97.7817 156.21 0)
       (effects (font (size 1.27 1.27)))
     )
@@
       (project "TAITOSJ"
         (path "/c9398d89-67dd-4ff5-9367-82e2b6879830/fa5496c1-bb75-4748-8ec7-34a2f42bf7c1"
-          (reference "U?") (unit 3)
+          (reference "U72") (unit 3)
         )
       )

Commit message: Tidied up loose ends
Connections:
- net LNSL1 is gone; now on net ~{LNSL1}: U2.1 (S)
- net OBJH is gone; now on net ~{OBJH}: U13.1 (S)
- net line_clock: now reaches U39.9, U7.5 (Q)
- net 8HN renamed 8HN'
Changed lines of the file:
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@@
     (effects (font (size 1.27 1.27)) (justify right bottom))
+  )
+  (label "line_clock" (at 394.97 210.82 0) (fields_autoplaced)
+    (effects (font (size 1.27 1.27)) (justify left bottom))
   )
   (label "Q22" (at 277.2376 180.34 0) (fields_autoplaced)
@@
     (effects (font (size 1.27 1.27)) (justify left bottom))
   )
-  (label "8HN" (at 346.71 213.36 0) (fields_autoplaced)
+  (label "8HN'" (at 346.71 213.36 0) (fields_autoplaced)
     (effects (font (size 1.27 1.27)) (justify left bottom))
   )
@@
     )
   )
-  (global_label "LNSL1" (shape input) (at 194.31 374.65 180) (fields_autoplaced)
-    (effects (font (size 1.27 1.27)) (justify right))
-    (property "Intersheetrefs" "${INTERSHEET_REFS}" (at 186.0912 374.5706 0)
+  (global_label "~{LNSL1}" (shape input) (at 194.31 374.65 180) (fields_autoplaced)
+    (effects (font (size 1.27 1.27)) (justify right))
+    (property "Intersheetrefs" "${INTERSHEET_REFS}" (at 185.5985 374.65 0)
       (effects (font (size 1.27 1.27)) (justify right) hide)
     )
@@
     )
   )
-  (global_label "OBJH" (shape input) (at 194.31 152.4 180) (fields_autoplaced)
+  (global_label "~{OBJH}" (shape input) (at 194.31 152.4 180) (fields_autoplaced)
     (effects (font (size 1.27 1.27)) (justify right))
     (property "Intersheetrefs" "${INTERSHEET_REFS}" (at 186.5056 152.4 0)

Commit message: Added MCU to Taito SJ Schematics
Parts:
- added U110: 74LS74, symbol jt74:74LS74
- added unit 5 of U4
- added unit 2 of U5
Connections:
- net CLK2: now also U110.11 (C), U110.3 (C)
- net H.INV: now also U110.1 (~{R}), U110.13 (~{R})
- net VCC: now also U110.10 (~{S}), U110.4 (~{S}), U5.10 (~{S}), U5.13 (~{R})
- net at U5.2 (D), U6.10, U6.5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: now also U5.12 (D)
- net at U19.6, U5.3 (C): now also U4.11
- new net: U110.2 (D), U5.9 (Q)
- new net: U4.10, U5.11 (C)
- new net: U110.12 (D), U5.8 (~{Q})
- new net ~{LNSL1X}: U110.5 (Q)
- new net ~{LNSL2X}: U110.9 (Q)
Other:
- note added: "ONLY ON FRONTLINE"
- moved on the sheet: U19B, U39C, U39D, U40, U54A, U54C, U5A, U6A, U6B, U6C, U6D, U7A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
