File: Taito System SJ/KiCAD/kscpu1.kicad_sch (KiCad schematic)
At the start: 116 parts

Commit message: Update kscpu1.kicad_sch
Parts:
- renumbered JKS_P to JKS_P1, JKS_Q to JKS_Q1
Connections:
- net ~{KSCPU_D0} is gone; now on net KSTIMER: UKS102.1 (SEL), UKS103.1, UKS58.12, UKS75.1 (SEL), UKS76.1 (SEL), UKS87.1 (SEL)
- net KSCPU_D0 renamed KSTIMER
Changed lines of the file:
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@@
 		)
 	)
-	(global_label "KSCPU_D0"
+	(global_label "KSTIMER"
 		(shape input)
 		(at 289.56 631.19 180)
@@
 		)
 		(property "Intersheetrefs" "${INTERSHEET_REFS}"
-			(at 276.7777 631.19 0)
+			(at 278.6525 631.19 0)
 			(effects
 				(font
@@
 		)
 	)
-	(global_label "~{KSCPU_D0}"
+	(global_label "KSTIMER"
 		(shape output)
 		(at 369.57 565.785 0)
@@
 		)
 		(property "Intersheetrefs" "${INTERSHEET_REFS}"
-			(at 382.3523 565.785 0)
+			(at 380.4775 565.785 0)
 			(effects
 				(font
@@
 		(dnp no)
 		(fields_autoplaced yes)
-		(property "Reference" "JKS_Q"
+		(property "Reference" "JKS_Q1"
 			(at 1143 100.965 0)
 			(effects
@@
 			(project ""
 				(path "/c9398d89-67dd-4ff5-9367-82e2b6879830/6fc72451-9f53-469a-bd1c-38914c38ced4"
-					(reference "JKS_Q")
+					(reference "JKS_Q1")
 					(unit 1)
 				)
@@
 		(dnp no)
 		(fields_autoplaced yes)
-		(property "Reference" "JKS_P"
+		(property "Reference" "JKS_P1"
 			(at 1143.635 22.225 0)
 			(effects
@@
 			(project "TAITOSJ"
 				(path "/c9398d89-67dd-4ff5-9367-82e2b6879830/6fc72451-9f53-469a-bd1c-38914c38ced4"
-					(reference "JKS_P")
+					(reference "JKS_P1")
 					(unit 1)
 				)
