File: Exidy440/KiCAD/mastercontrol.kicad_sch (KiCad schematic)
At the start: 35 parts, among them U10H 74LS161, U10L 74LS32, U11H 74LS161, U12H LS287, U13H 74LS161, U14H 74LS161, U23B 74LS25, U23D 74LS08, U2K 74LS112, U2L 74LS04, U3K MB7112E, U3L 74LS86, U4K LS287, U5J 74LS04, U5K LS287, U5L 74LS374, U6H 74LS04, U6J 74LS161, U6K LS287, U6L 74LS374, U7J 74LS161, U7K LS287, U7L 74LS374, U8J 74LS153, U8K LS287, U8L 74LS374, U9H LS287, U9J 74LS74, U9L 74LS08

Commit message: Misc fixes found while checking clocks in FPGA core
Parts:
- added unit 4 of U5J
Connections:
- net +5V: now also U6J.1 (~{MR}), U6J.10 (CET), U6J.3 (D0), U6J.4 (D1), U6J.5 (D2), U6J.6 (D3), U6J.7 (CEP), U6J.9 (~{PE}), U7J.1 (~{MR})
- net C3: now also U8L.17 (D6), U5J.9
- net GND: now also U9H.1 (A6), U9H.13 (~{CS0}), U9H.14 (~{CS1}), U9H.15 (A7)
- net at U8L.18 (D7): now also U5J.8
- net $D0 renamed S=0
Other:
- note removed: "Check this is really $D0"
- moved on the sheet: U10LC, U8L, U9LC

Commit message: Added dual PCB structure, misc fixes and start of audio board IO
Parts:
- renumbered 12.9792MHz to 12.9792MHz?, E1 to E?, R3 to R?, U10H to U10H?, U10L to U10L?, U11H to U11H?, U12H to U12H?, U13H to U13H?, U14H to U14H?, U23B to U23B?, U23D to U23D?, U2K to U2K?, U2L to U2L?, U3K to U3K?, U3L to U3L?, U4K to U4K?, U5J to U5J?, U5K to U5K?, U5L to U5L?, U6H to U6H?, U6J to U6J?, U6K to U6K?, U6L to U6L?, U7J to U7J?, U7K to U7K?, U7L to U7L?, U8J to U8J?, U8K to U8K?, U8L to U8L?, U9H to U9H?, U9J to U9J?, U9L to U9L?
Other:
- note added: "0.8112Mhz"
- note added: "1.6224Mhz"
- note added: "12.9792MHz"
- note added: "3.2448Mhz"
- note added: "6.4896Mhz"

Commit message: Correction of references after copy/paste issue.  Additional IO on audio board.
Parts:
- Y1: renamed from 12.9792MHz?; value Y1 -> 12.9792MHz
- gave numbers to parts that had none: 31
