File: Exidy440/KiCAD/video.kicad_sch (KiCad schematic)
At the start: 54 parts, among them P3 Power Connector, P4 Video Output, Q1 2N3904, Q2 2N3906, Q3 2N3904, Q4 2N3906, Q5 2N3904, Q6 2N3906, Q7 2N3904, U19K 74LS05, U20K 74LS05, U21K 74LS05, U22K 74LS86

Commit message: Added dual PCB structure, misc fixes and start of audio board IO
Parts:
- renumbered C1C to C1C?, C8 to C?, C7 to C?, C5 to C?, C6 to C?, CR4 to CR?, CR2 to CR?, CR3 to CR?, CR5 to CR?, E3 to E?, P3 to P?, P4 to P?, Q1 to Q?, Q4 to Q?, Q5 to Q?, Q7 to Q?, Q2 to Q?, Q3 to Q?, Q6 to Q?, R40 to R?, R37 to R?, R42 to R?, R38 to R?, R28 to R?, R50 to R?, R48 to R?, R46 to R?, R22 to R?, R35 to R?, R44 to R?, R31 to R?, R39 to R?, R43 to R?, R26 to R?, R25 to R?, R29 to R?, R49 to R?, R45 to R?, R33 to R?, R24 to R?, R21 to R?, R41 to R?, R34 to R?, R32 to R?, R30 to R?, R47 to R?, R27 to R?, R23 to R?, U19K to U19K?, U20K to U20K?, U21K to U21K?, U22K to U22K?, VR1 to VR?

Commit message: Correction of references after copy/paste issue.  Additional IO on audio board.
Parts:
- gave numbers to parts that had none: 53
