File: Exidy440/KiCAD/vramseq.kicad_sch (KiCad schematic)
At the start: 50 parts, among them U13B 74LS245, U13C 74LS245, U13D 74LS245, U13E 74LS245, U13F 74LS139, U14A 74LS166, U14B HM6116P-3, U14C HM6116P-3, U14D HM6116P-3, U14E HM6116P-3, U14F 74LS138, U15A 74LS166, U15F 74LS151, U15H 74LS151, U16A 74LS166, U16B HM6116P-3, U16C HM6116P-3, U16D HM6116P-3, U16E HM6116P-3, U16F 74LS151, U16H 74LS151, U17A 74LS166, U17B HM6116P-3, U17C HM6116P-3, U17D HM6116P-3, U17E HM6116P-3, U17F 74LS151, U17H 74LS151, U18B HM6116P-3, U18C HM6116P-3, U18D HM6116P-3, U18E HM6116P-3, U18F 74LS151, U18H 74LS151, U19F 74LS151, U19H 74LS151, U20B HM6116P-3, U20C HM6116P-3, U20D HM6116P-3, U20E HM6116P-3, U20F 74LS151, U20H 74LS151, U21B HM6116P-3, U21C HM6116P-3, U21D HM6116P-3, U21E HM6116P-3, U21F 74LS151, U21H 74LS151, U23E 74LS374, U6H 74LS04

Commit message: Added dual PCB structure, misc fixes and start of audio board IO
Parts:
- renumbered U13B to U13B?, U13C to U13C?, U13D to U13D?, U13E to U13E?, U13F to U13F?, U14A to U14A?, U14B to U14B?, U14C to U14C?, U14D to U14D?, U14E to U14E?, U14F to U14F?, U15A to U15A?, U15F to U15F?, U15H to U15H?, U16A to U16A?, U16B to U16B?, U16C to U16C?, U16D to U16D?, U16E to U16E?, U16F to U16F?, U16H to U16H?, U17A to U17A?, U17B to U17B?, U17C to U17C?, U17D to U17D?, U17E to U17E?, U17F to U17F?, U17H to U17H?, U18B to U18B?, U18C to U18C?, U18D to U18D?, U18E to U18E?, U18F to U18F?, U18H to U18H?, U19F to U19F?, U19H to U19H?, U20B to U20B?, U20C to U20C?, U20D to U20D?, U20E to U20E?, U20F to U20F?, U20H to U20H?, U21B to U21B?, U21C to U21C?, U21D to U21D?, U21E to U21E?, U21F to U21F?, U21H to U21H?, U23E to U23E?, U6H to U6H?

Commit message: Correction of references after copy/paste issue.  Additional IO on audio board.
Parts:
- gave numbers to parts that had none: 50
