File: Exidy440/KiCAD/logicvideo.kicad_sch (KiCad schematic)
At the start: 0 parts

Commit message: Minor modifications to IO board
Other:
- sheet Video Out renamed Power Connector & Video Out
Changed lines of the file:
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@@
 			(color 0 0 0 0.0000)
 		)
-		(property "Sheetname" "Video Out"
+		(property "Sheetname" "Power Connector & Video Out"
 			(at 228.6 24.6884 0)
 			(effects
