File: ExidyUGB2/exidy2/TAUDIO2.kicad_sch (KiCad schematic)
At the start: 74 parts, among them Q4 2N3904, U3C_ 74LS04, U4A MC3340, U4B LM566, U4C_ 74LS07, U5A_ LM556, U5B_ LM324, U6A_ LM379

Commit message: Updates to KiCAD8
Parts:
- renumbered C49 to C10, C46 to C11, C42 to C12, C46 to C13, C46 to C14, C49 to C15, C42 to C16, C46 to C26, C49 to C28, C46 to C29, C42 to C31, C42 to C32, C42 to C34, C46 to C35, C46 to C36, C42 to C37, C42 to C38, C42 to C39, C46 to C40, C49 to C5, C46 to C50, C49 to C7, C49 to C9, CR4 to CR1, CR4 to CR2, CR4 to CR3, Q4 to Q1, Q4 to Q2, Q4 to Q3, R23 to R1, R23 to R10, R45 to R11, R36 to R12, R41 to R13, R41 to R14, R41 to R18, R36 to R19, R45 to R2, R41 to R20, R36 to R21, R46 to R24, R45 to R25, R36 to R26, R36 to R27, R46 to R28, R23 to R29, R45 to R3, R36 to R30, R36 to R31, R46 to R32, R45 to R33, R46 to R34, R23 to R35, R46 to R39, R45 to R4, R36 to R49, R45 to R5, R36 to R50, R41 to R6, R41 to R7, R41 to R8, R41 to R9, R23 to R?
