File: Exerion/KiCAD/CPUB.kicad_sch (KiCad schematic)
At the start: 68 parts, among them U2S1 74LS374, U3A1 74LS191, U3B1 74LS374, U3C1 74LS374, U3D1 74LS191, U3D2 6301, U3E1 74LS191, U3F1 74LS374, U3H1 74LS374, U3J1 74LS191, U3K1 74LS374, U3T1 74LS138, U4B1 2764, U4D1 2764, U4E1 2764, U4H1 2764, U4KJ1 6301, U4LK_1 74LS32, U4ML1 74LS153, U4T1 2764, U4V1 HM6116P-3, U5,6V1 Z80CPUB, U5A1 74LS153, U5B1 74LS374, U5C1 74LS153, U5D1 74LS374, U5E1 74LS374, U5F1 74LS153, U5H1 74LS374, U5J1 74LS153, U5ST_1 74LS04, U5UT1 74LS89, U6A1 74LS193, U6B1 74LS191, U6C1 74LS191, U6D1 74LS193, U6E1 74LS193, U6F1 74LS191, U6H1 74LS191, U6J1 74LS193, U6ST_1 74LS04, U6UT1 74LS89, U7A1 74LS74, U7A_1 74LS74, U7B_1 74LS86, U7D_1 74LS74, U7E_1 74LS74, U7F_1 74LS08, U7H_1 74LS86, U7J_1 74LS74, U7V1 74LS157, U8A1 74LS193, U8B1 74LS193, U8C1 74LS193, U8D1 74LS193, U8E1 74LS138, U8H2 74LS138, U8T_1 74LS74, U8U_1 74LS125, U9C_1 74LS04, U9C_2 74LS04, U9D_1 74LS32, U9U_1 74LS86, U9_C1 74LS04, U9_D1 74LS32, U9_P1 74LS04

Commit message: Component naming updates
Connections:
- net L4B_clk2: now reaches U5B1.11 (Cp), U7A_1.11 (C), U7B_1.3
- net L4B_clk1: now reaches U6A1.5 (CpUp), U7B_1.6, U8A1.5 (CpUp)

Commit message: Exerion Updates to KiCAD 8
Parts:
- removed U9U_1: 74LS86, symbol jt74:74LS86
- added R?: 1K, symbol Device:R_US
- added U7U_: 74LS32, symbol 74xx:74LS32
Connections:
- net GNDPWR: now also U3A1.4 (~{CEN}), U3B1.1 (~{OE}), U3C1.1 (~{OE}), U3D1.4 (~{CEN}), U3E1.4 (~{CEN}), U3F1.1 (~{OE}), U3H1.1 (~{OE}), U3J1.4 (~{CEN}), U7V1.15 (E)
- net SSEL: now also U7V1.1 (S); no longer U9D_1.4
- net VCC: now also R?.1
- net at U9C_1.2, U9_D1.2: now also U9D_1.4
- net at U3T1.11 (O4): now also U7U_.5
- net at U4V1.21 (~{WR}), U5,6V1.22 (~{WR}): now also U7U_.4
- net at U5UT1.3 (~{WE}), U6UT1.3 (~{WE}): now also U7U_.6
- net at U5,6V1.16 (~{INT}), U5,6V1.17 (~{NMI}), U5,6V1.24 (~{WAIT})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: now also R?.2
